File: PCB/Remote_Weather_Station/Remote_Weather_Station.kicad_sch (KiCad schematic)
At the start: 25 parts, among them J101 strain_gauge_N, J102 strain_gauge_E, J103 strain_gauge_S, J104 strain_gauge_W, J105 load_cell_in, J106 UART, J107 Stemma_QT_Connector, J108 Servo_Connector, SW101 SW_Push, SW102 SW_Push, U101 ESP32-WROOM-32D

Commit message: Add files via upload
Parts:
- removed J101: strain_gauge_N, symbol Connector_Generic:Conn_01x02
- removed J102: strain_gauge_E, symbol Connector_Generic:Conn_01x02
- removed J103: strain_gauge_S, symbol Connector_Generic:Conn_01x02
- removed J104: strain_gauge_W, symbol Connector_Generic:Conn_01x02
- removed J105: load_cell_in, symbol Connector_Generic:Conn_01x02
- removed R101, R102: 350, symbol Device:R_Small_US
- added C104, C105, C107, C108, C109, C110, C111, C112: 1u, Capacitor_SMD:C_0805_2012Metric, symbol Device:C_Small
- added H101, H102, H103, H104: MountingHole, MountingHole:MountingHole_3.2mm_M3, symbol Mechanical:MountingHole
- added J103: wire_bus, symbol Connector_Generic:Conn_01x12
- added J105: power_in, symbol Connector_Generic:Conn_01x04
- added R107: 20, Resistor_SMD:R_0402_1005Metric, symbol Device:R_Small_US
- added R108: 330, Resistor_SMD:R_0402_1005Metric, symbol Device:R_Small_US
- added R110, R111: 2k, Resistor_SMD:R_0402_1005Metric, symbol Device:R_Small_US
- added R112, R113, R117: 11k, Resistor_SMD:R_0402_1005Metric, symbol Device:R_Small_US
- added R114, R115, R118: 4.7k, Resistor_SMD:R_0402_1005Metric, symbol Device:R_Small_US
- added R116: 82, Resistor_SMD:R_0402_1005Metric, symbol Device:R_Small_US
- added U102, U103, U104: AD8227, Package_SO:SOIC-8_3.9x4.9mm_P1.27mm, symbol Amplifier_Instrumentation:AD8236
- C101: footprint (none) -> Capacitor_SMD:C_0805_2012Metric; JLCPCB# (none) -> C49678
- C102, C103: value 1uF -> 1u; footprint (none) -> Capacitor_SMD:C_0805_2012Metric; JLCPCB# (none) -> C28323
- C106: renamed from C105; value 1uF -> 1u; footprint (none) -> Capacitor_SMD:C_0805_2012Metric; JLCPCB# (none) -> C28323
- D101: footprint (none) -> LED_SMD:LED_0805_2012Metric_Pad1.15x1.40mm_HandSolder
- J101: renamed from J106; now left out of the parts list
- R101: renamed from R115; footprint (none) -> Resistor_SMD:R_0402_1005Metric
- R102: renamed from R105; value 12k -> 4.7k; footprint (none) -> Resistor_SMD:R_0402_1005Metric
- R103: value 350 -> 20; footprint (none) -> Resistor_SMD:R_0402_1005Metric
- R104: value 350 -> 330; footprint (none) -> Resistor_SMD:R_0402_1005Metric
- R105: renamed from R113; footprint (none) -> Resistor_SMD:R_0402_1005Metric
- R106: renamed from R114; footprint (none) -> Resistor_SMD:R_0402_1005Metric
- R109: renamed from R116; value 12k -> 4.7k; footprint (none) -> Resistor_SMD:R_0402_1005Metric
- renumbered J107 to J102, J108 to J104, SW102 to SW101, SW101 to SW102
Connections:
- net +3.3V: now also C104.2, C105.2, C107.1, J103.1 (Pin_1), J103.3 (Pin_3), J103.9 (Pin_9); no longer R104.1
- net +5V: now also C108.2, C109.2, C110.2, C111.1, C112.1, R112.1, R113.1, R117.1, U102.8 (Vs+), U103.8 (Vs+), U104.8 (Vs+)
- net GND: now also C104.1, C105.1, C107.2, C108.1, C109.1, C110.1, C111.2, C112.2, J103.12 (Pin_12), J103.6 (Pin_6), J103.8 (Pin_8), J105.2 (Pin_2), J105.4 (Pin_4), R108.2, R114.2, R115.2, R118.2, U102.5 (Vs-), U103.5 (Vs-), U104.5 (Vs-)
- net Green_Wire: now also J103.10 (Pin_10), U104.1 (-)
- net Servo: now also U101.30 (IO18); no longer U101.37 (IO23)
- net White_Wire: now also J103.11 (Pin_11), U104.4 (+)
- net East_Test renamed E_W_Value
- net E_W_Value: now also U103.7
- net North_Test renamed N_S_Value
- net N_S_Value: now also U102.7
- net South_Test: no longer names the net of R103.2
- net South_Test: now also R104.2; no longer U101.13 (IO14)
- net Vwater: no longer names the net of U101.27 (IO16)
- net West_Test: no longer names the net of U101.23 (IO15)
- net West_Test: no longer R104.2
- new net: R113.2, R115.1, U103.6 (Ref)
- new net: R112.2, R114.1, U102.6 (Ref)
- new net: R110.1, U102.2 (Rg)
- new net: R110.2, U102.3 (Rg)
- new net: R111.1, U103.2 (Rg)
- new net: R111.2, U103.3 (Rg)
- new net: R117.2, R118.1, U104.6 (Ref)
- new net: R116.1, U104.2 (Rg)
- new net: R116.2, U104.3 (Rg)
- new net: R107.2, R108.1
- new net +12V: J105.1 (Pin_1)
- new net +5V_panel: J105.3 (Pin_3)
- new net Base_Ref: R104.1, R107.1, U102.1 (-), U103.1 (-)
- new net East_West_Ref: J103.4 (Pin_4), J103.7 (Pin_7), U103.4 (+)
- new net North_South_Ref: J103.2 (Pin_2), J103.5 (Pin_5), U102.4 (+)
- new net Rain_Value: U101.13 (IO14), U104.7
- no-connect marks 0 -> 8
Other:
- added sheet PDN (PDN.kicad_sch)
- note added: "Analog Sensors Anemometer Precipitation"
- note added: "Analog Sensors Instrumentation Amps"
- note added: "Double Check gain resistors"
- note added: "Microcontroller ESP32"
- note added: "PDN and Input Power"
- note added: "Precipitation Drainage Servo"
- note added: "Sensor Bus I2C Communication Bus"
- note added: "load_cell black_wire"
- note added: "load_cell red_wire"
- note removed: "Anemometer Strain Gauges"
- note removed: "ESP32"
- note removed: "Instrumentation Amplifier Setup"
- note removed: "Rain Gauge Loadcell"
- note removed: "Rain Gauge Servo Control"
- note removed: "Sensors I2C Communication Bus"
- moved on the sheet: J104

Commit message: Add files via upload
Parts:
- R110, R111: value 2k -> 16k
Changed lines of the file:
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@@
 			)
 		)
-		(property "Value" "2k"
+		(property "Value" "16k"
 			(at 88.9 170.1799 0)
 			(effects
@@
 			)
 		)
-		(property "Value" "2k"
+		(property "Value" "16k"
 			(at 146.05 170.1799 0)
 			(effects

Commit message: Add files via upload
Other:
- note added: ""Boot""
Changed lines of the file:
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@@
+		)
+	)
+	(text "\"Boot\""
+		(exclude_from_sim no)
+		(at 92.456 50.8 0)
+		(effects
+			(font
+				(size 1.27 1.27)
+			)
+			(justify left)
 		)
 	)

Commit message: Add files via upload
Parts:
- added C113: 1u, Capacitor_SMD:C_0805_2012Metric, symbol Device:C_Small
Connections:
- net Flash: now also C113.1
- net GND: now also C113.2
Other:
- title: Remote Weather Station -> Weather Station
Changed lines of the file:
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@@
 	(paper "A4")
 	(title_block
-		(title "Remote Weather Station")
+		(title "Weather Station")
 		(date "2026-01-22")
 		(rev "V1")
@@
 	)
 	(junction
+		(at 116.84 110.49)
+		(diameter 0)
+		(color 0 0 0 0)
+	)
+	(junction
 		(at 239.395 86.36)
 		(diameter 0)
@@
 	(wire
 		(pts
+			(xy 116.84 118.11) (xy 116.84 120.65)
+		)
+		(stroke
+			(width 0)
+			(type default)
+		)
+	)
+	(wire
+		(pts
 			(xy 165.1 124.46) (xy 165.1 127)
 		)
@@
 	(wire
 		(pts
+			(xy 116.84 110.49) (xy 116.84 113.03)
+		)
+		(stroke
+			(width 0)
+			(type default)
+		)
+	)
+	(wire
+		(pts
 			(xy 176.53 180.34) (xy 176.53 177.8)
 		)
@@
 		)
 	)
+	(wire
+		(pts
+			(xy 116.84 110.49) (xy 120.65 110.49)
+		)
+		(stroke
+			(width 0)
+			(type default)
+		)
+	)
 	(label "E_red_wire"
 		(at 257.175 73.66 180)
@@
 	(global_label "Flash"
 		(shape bidirectional)
-		(at 116.84 110.49 0)
+		(at 120.65 110.49 0)
 		(fields_autoplaced yes)
 		(effects
@@
 		)
 		(property "Intersheetrefs" "${INTERSHEET_REFS}"
-			(at 126.0164 110.49 0)
+			(at 129.8264 110.49 0)
 			(effects
 				(font
@@
 	)
 	(symbol
+		(lib_id "Device:C_Small")
+		(at 116.84 115.57 0)
+		(unit 1)
+		(exclude_from_sim no)
+		(in_bom yes)
+		(on_board yes)
+		(dnp no)
+		(fields_autoplaced yes)
+		(property "Reference" "C113"
+			(at 119.38 114.3062 0)
+			(effects
+				(font
+					(size 1.27 1.27)
+				)
+				(justify left)
+			)
+		)
+		(property "Value" "1u"
+			(at 119.38 116.8462 0)
+			(effects
+				(font
+					(size 1.27 1.27)
+				)
+				(justify left)
+			)
+		)
+		(property "Footprint" "Capacitor_SMD:C_0805_2012Metric"
+			(at 116.84 115.57 0)
+			(effects
+				(font
+					(size 1.27 1.27)
+				)
+				(hide yes)
+			)
+		)
+		(property "Datasheet" "~"
+			(at 116.84 115.57 0)
+			(effects
+				(font
+					(size 1.27 1.27)
+				)
+				(hide yes)
+			)
+		)
+		(property "Description" "Unpolarized capacitor, small symbol"
+			(at 116.84 115.57 0)
+			(effects
+				(font
+					(size 1.27 1.27)
+				)
+				(hide yes)
+			)
+		)
+		(property "JLCPCB#" "C28323"
+			(at 116.84 115.57 0)
+			(effects
+				(font
+					(size 1.27 1.27)
+				)
+				(hide yes)
+			)
+		)
+		(pin "2"
+		)
+		(pin "1"
+		)
+		(instances
+			(project "Remote_Weather_Station"
+				(path "/a9f3e948-f0cb-4784-bed2-bdf72b5832ff"
+					(reference "C113")
+					(unit 1)
+				)
+			)
+		)
+	)
+	(symbol
 		(lib_id "Amplifier_Instrumentation:AD8236")
 		(at 162.56 168.91 0)
@@
 					(unit 1)
 				)
+			)
+		)
+	)
+	(symbol
+		(lib_id "power:GND")
+		(at 116.84 120.65 0)
+		(unit 1)
+		(exclude_from_sim no)
+		(in_bom yes)
+		(on_board yes)
+		(dnp no)
+		(fields_autoplaced yes)
+		(property "Reference" "#PWR0155"
+			(at 116.84 127 0)
+			(effects
+				(font
+					(size 1.27 1.27)
+				)
+				(hide yes)
+			)
+		)
+		(property "Value" "GND"
+			(at 116.84 125.73 0)
+			(effects
+				(font
+					(size 1.27 1.27)
+				)
+				(hide yes)
+			)
+		)
+		(property "Footprint" ""
+			(at 116.84 120.65 0)
+			(effects
+				(font
+					(size 1.27 1.27)
+				)
+				(hide yes)
+			)
+		)
+		(property "Datasheet" ""
+			(at 116.84 120.65 0)
+			(effects
+				(font
+					(size 1.27 1.27)
+				)
+				(hide yes)
+			)
+		)
+		(property "Description" "Power symbol creates a global label with name \"GND\" , ground"
+			(at 116.84 120.65 0)
+			(effects
+				(font
+					(size 1.27 1.27)
+				)
+				(hide yes)
+			)
+		)
+		(pin "1"
+		)
+		(instances
+			(project "Remote_Weather_Station"
+				(path "/a9f3e948-f0cb-4784-bed2-bdf72b5832ff"
+					(reference "#PWR0155")
+					(unit 1)
+				)

Commit message: Add files via upload
Parts:
- removed R113: 11k, Resistor_SMD:R_0402_1005Metric, symbol Device:R_Small_US
- removed R115: 4.7k, Resistor_SMD:R_0402_1005Metric, symbol Device:R_Small_US
- added C114, C115, C116: 1u, Capacitor_SMD:C_0805_2012Metric, symbol Device:C_Small
- added R116, R121: 1k, Resistor_SMD:R_0603_1608Metric_Pad0.98x0.95mm_HandSolder, symbol Device:R_Small_US
- added R117: 10k, Resistor_SMD:R_0603_1608Metric_Pad0.98x0.95mm_HandSolder, symbol Device:R_Small_US
- added R119, R120: 4.7k, Resistor_SMD:R_0603_1608Metric_Pad0.98x0.95mm_HandSolder, symbol Device:R_Small_US
- D101: value LED -> RED_LED; footprint LED_SMD:LED_0805_2012Metric_Pad1.15x1.40mm_HandSolder -> LED_SMD:LED_0603_1608Metric; JLCPCB# (none) -> C2286
- J102: JLCPCB# (none) -> C160404
- R101: footprint Resistor_SMD:R_0402_1005Metric -> Resistor_SMD:R_0603_1608Metric_Pad0.98x0.95mm_HandSolder; JLCPCB# (none) -> C23228
- R102, R105, R106, R118: footprint Resistor_SMD:R_0402_1005Metric -> Resistor_SMD:R_0603_1608Metric_Pad0.98x0.95mm_HandSolder; JLCPCB# (none) -> C23162
- R103, R107: footprint Resistor_SMD:R_0402_1005Metric -> Resistor_SMD:R_0603_1608Metric_Pad0.98x0.95mm_HandSolder; JLCPCB# (none) -> C22950
- R104, R108: footprint Resistor_SMD:R_0402_1005Metric -> Resistor_SMD:R_0603_1608Metric_Pad0.98x0.95mm_HandSolder; JLCPCB# (none) -> C23138
- R109: footprint Resistor_SMD:R_0402_1005Metric -> Resistor_SMD:R_0603_1608Metric_Pad0.98x0.95mm_HandSolder; JLCPCB# C21190 -> C23162
- R110: renamed from R116; value 82 -> 100; footprint Resistor_SMD:R_0402_1005Metric -> Resistor_SMD:R_0603_1608Metric_Pad0.98x0.95mm_HandSolder; JLCPCB# (none) -> C22775
- R111: renamed from R110; value 16k -> 15k; footprint Resistor_SMD:R_0402_1005Metric -> Resistor_SMD:R_0603_1608Metric_Pad0.98x0.95mm_HandSolder; JLCPCB# (none) -> C22809
- R112: renamed from R111; value 16k -> 15k; footprint Resistor_SMD:R_0402_1005Metric -> Resistor_SMD:R_0603_1608Metric_Pad0.98x0.95mm_HandSolder; JLCPCB# (none) -> C22809
- R113: renamed from R117; value 11k -> 10k; footprint Resistor_SMD:R_0402_1005Metric -> Resistor_SMD:R_0603_1608Metric_Pad0.98x0.95mm_HandSolder; JLCPCB# (none) -> C25804
- R114: value 4.7k -> 1k; footprint Resistor_SMD:R_0402_1005Metric -> Resistor_SMD:R_0603_1608Metric_Pad0.98x0.95mm_HandSolder; JLCPCB# (none) -> C21190
- R115: renamed from R112; value 11k -> 10k; footprint Resistor_SMD:R_0402_1005Metric -> Resistor_SMD:R_0603_1608Metric_Pad0.98x0.95mm_HandSolder; JLCPCB# (none) -> C25804
- U101: JLCPCB# (none) -> C473012
- U102: renamed from U104; JLCPCB# (none) -> C652556
- U103: renamed from U102; JLCPCB# (none) -> C652556
- U104: renamed from U103; JLCPCB# (none) -> C652556
- renumbered C104 to C101, C105 to C102, C101 to C103, C102 to C104, C103 to C105, C111 to C107, C107 to C108, C112 to C109, C113 to C110, C108 to C111, C109 to C112, C110 to C113
Connections:
- net +5V: now also R114.1, R116.1, R121.1; no longer R113.1, R115.1
- net GND: now also C114.1, C115.1, C116.1, R119.2, R120.2; no longer R114.2
- net at U104.6 (Ref): now also C116.2, R117.2, R120.1
- net at R115.2, U103.6 (Ref): now also C115.2, R119.1; no longer R114.1
- net at R113.2, R118.1, U102.6 (Ref): now also C114.2
- new net: R117.1, R121.2
- new net: R115.1, R116.2
- new net: R113.1, R114.2
Other:
- moved on the sheet: R111, R112, R118

Commit message: Add files via upload
Parts:
- added C117: 1u, Capacitor_SMD:C_0805_2012Metric, symbol Device:C_Small
- added U105: SIM7600X, symbol ModemSymbol:Modem_Sym
- R110: value 100 -> 820
Connections:
- net +5V_panel: now also C117.1, U105.19 (VIN)
- net GND: now also C117.2, U105.10 (GND), U105.18 (GND), U105.26 (GND)
Other:
- note added: "Modem"

Commit message: Add files via upload
Parts:
- R110: JLCPCB# C22775 -> (none)
Changed lines of the file:
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@@
 			)
 		)
-		(property "JLCPCB#" "C22775"
+		(property "JLCPCB#" ""
 			(at 25.4 168.91 0)
 			(effects

Commit message: Add files via upload
Parts:
- H101, H102, H103, H104: footprint MountingHole:MountingHole_3.2mm_M3 -> MountingHole:MountingHole_2.7mm_M2.5
- J101: footprint (none) -> Connector_PinHeader_2.54mm:PinHeader_1x06_P2.54mm_Vertical
- J102: footprint (none) -> Connector_JST:JST_SH_BM04B-SRSS-TB_1x04-1MP_P1.00mm_Vertical
- J103: footprint (none) -> Terminal_Blocks:WJ250B-3.5-12P-11-00A
- J104: footprint (none) -> Connector_PinHeader_2.54mm:PinHeader_1x03_P2.54mm_Vertical
- J105: footprint (none) -> Terminal_Blocks:DBT50G-7.62-4P-BK-P
- R110: JLCPCB# (none) -> C23253
- SW101, SW102: footprint button:TS-1088-AR02016 -> Button_Switch_SMD:SW_SPST_TS-1088-xR020
- U105: footprint (none) -> Modem_Footprint:SIM7600X
Changed lines of the file:
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@@
 			)
 		)
-		(property "Footprint" "MountingHole:MountingHole_3.2mm_M3"
+		(property "Footprint" "MountingHole:MountingHole_2.7mm_M2.5"
 			(at 17.78 129.54 0)
 			(effects
@@
 			)
 		)
-		(property "Footprint" ""
+		(property "Footprint" "Terminal_Blocks:DBT50G-7.62-4P-BK-P"
 			(at 172.72 119.38 0)
 			(effects
@@
 			)
 		)
-		(property "Footprint" "MountingHole:MountingHole_3.2mm_M3"
+		(property "Footprint" "MountingHole:MountingHole_2.7mm_M2.5"
 			(at 17.78 116.84 0)
 			(effects
@@
 			)
 		)
-		(property "Footprint" ""
+		(property "Footprint" "Connector_JST:JST_SH_BM04B-SRSS-TB_1x04-1MP_P1.00mm_Vertical"
 			(at 151.13 64.77 0)
 			(effects
@@
 			)
 		)
-		(property "Footprint" ""
+		(property "Footprint" "Terminal_Blocks:WJ250B-3.5-12P-11-00A"
 			(at 264.795 78.74 0)
 			(effects
@@
 			)
 		)
-		(property "Footprint" "MountingHole:MountingHole_3.2mm_M3"
+		(property "Footprint" "MountingHole:MountingHole_2.7mm_M2.5"
 			(at 17.78 110.49 0)
 			(effects
@@
 			)
 		)
+		(property "JLCPCB#" ""
+			(at 17.78 110.49 0)
+			(effects
+				(font
+					(size 1.27 1.27)
+				)
+				(hide yes)
+			)
+		)
 		(instances
 			(project ""
@@
 			)
 		)
-		(property "JLCPCB#" ""
+		(property "JLCPCB#" "C23253"
 			(at 25.4 168.91 0)
 			(effects
@@
 			)
 		)
-		(property "Footprint" "button:TS-1088-AR02016"
+		(property "Footprint" "Button_Switch_SMD:SW_SPST_TS-1088-xR020"
 			(at 106.68 105.41 0)
 			(effects
@@
 			)
 		)
-		(property "Footprint" ""
+		(property "Footprint" "Modem_Footprint:SIM7600X"
 			(at 228.6 157.48 0)
 			(effects
@@
 			)
 		)
+		(property "JLCPCB#" ""
+			(at 228.6 157.48 0)
+			(effects
+				(font
+					(size 1.27 1.27)
+				)
+				(hide yes)
+			)
+		)
 		(pin "13"
 		)
@@
 			)
 		)
-		(property "Footprint" ""
+		(property "Footprint" "Connector_PinHeader_2.54mm:PinHeader_1x06_P2.54mm_Vertical"
 			(at 143.51 31.75 0)
 			(effects
@@
 			)
 		)
-		(property "Footprint" ""
+		(property "Footprint" "Connector_PinHeader_2.54mm:PinHeader_1x03_P2.54mm_Vertical"
 			(at 158.75 90.17 0)
 			(effects
@@
 			)
 		)
-		(property "Footprint" "MountingHole:MountingHole_3.2mm_M3"
+		(property "Footprint" "MountingHole:MountingHole_2.7mm_M2.5"
 			(at 17.78 123.19 0)
 			(effects
@@
 			)
 		)
-		(property "Footprint" "button:TS-1088-AR02016"
+		(property "Footprint" "Button_Switch_SMD:SW_SPST_TS-1088-xR020"
 			(at 25.4 48.26 0)
 			(effects
