File: PCB/Remote_Weather_Station/Remote_Weather_Station.kicad_sch (KiCad schematic)
At the start: 40 parts, among them J101 UART, J102 Stemma_QT_Connector, J103 Servo_Connector, J104 load_cell_in, J105 strain_gauge_N, J106 strain_gauge_S, J107 strain_gauge_E, J108 strain_gauge_W, SW101 SW_Push, SW102 SW_Push, U101 AD8227, U102 ESP32-WROOM-32D, U103 AD8227, U104 AD8227

Commit message: Add files via upload
Laid out PDN
Parts:
- removed J104: load_cell_in, symbol Connector_Generic:Conn_01x04
- removed J105: strain_gauge_N, symbol Connector_Generic:Conn_01x02
- removed J106: strain_gauge_S, symbol Connector_Generic:Conn_01x02
- removed J107: strain_gauge_E, symbol Connector_Generic:Conn_01x02
- removed J108: strain_gauge_W, symbol Connector_Generic:Conn_01x02
- removed R103, R110: 4.7k, Resistor_SMD:R_0402_1005Metric, symbol Device:R_Small_US
- removed R112: 11k, Resistor_SMD:R_0402_1005Metric, symbol Device:R_Small_US
- added C107, C109, C110, C111, C112, C113, C114, C115, C116, C117: 1u, Capacitor_SMD:C_0805_2012Metric, symbol Device:C_Small
- added H101, H102, H103, H104: MountingHole, MountingHole:MountingHole_2.7mm_M2.5, symbol Mechanical:MountingHole
- added J103: wire_bus, Terminal_Blocks:WJ250B-3.5-12P-11-00A, symbol Connector_Generic:Conn_01x12
- added J105: power_in, Terminal_Blocks:DBT50G-7.62-4P-BK-P, symbol Connector_Generic:Conn_01x04
- added R114, R116, R121: 1k, Resistor_SMD:R_0603_1608Metric_Pad0.98x0.95mm_HandSolder, symbol Device:R_Small_US
- added R117: 10k, Resistor_SMD:R_0603_1608Metric_Pad0.98x0.95mm_HandSolder, symbol Device:R_Small_US
- added R119, R120: 4.7k, Resistor_SMD:R_0603_1608Metric_Pad0.98x0.95mm_HandSolder, symbol Device:R_Small_US
- added U105: SIM7600X, Modem_Footprint:SIM7600X, symbol ModemSymbol:Modem_Sym
- D101: value LED -> RED_LED; footprint (none) -> LED_SMD:LED_0603_1608Metric; JLCPCB# (none) -> C2286
- J101: footprint (none) -> Connector_PinHeader_2.54mm:PinHeader_1x06_P2.54mm_Vertical; now left out of the parts list
- J102: footprint (none) -> Connector_JST:JST_SH_BM04B-SRSS-TB_1x04-1MP_P1.00mm_Vertical; JLCPCB# (none) -> C160404
- J104: renamed from J103; footprint (none) -> Connector_PinHeader_2.54mm:PinHeader_1x03_P2.54mm_Vertical
- R101: renamed from R114; footprint Resistor_SMD:R_0402_1005Metric -> Resistor_SMD:R_0603_1608Metric_Pad0.98x0.95mm_HandSolder; JLCPCB# (none) -> C23228
- R102: footprint Resistor_SMD:R_0402_1005Metric -> Resistor_SMD:R_0603_1608Metric_Pad0.98x0.95mm_HandSolder; JLCPCB# (none) -> C23162
- R103: renamed from R115; footprint Resistor_SMD:R_0402_1005Metric -> Resistor_SMD:R_0603_1608Metric_Pad0.98x0.95mm_HandSolder; JLCPCB# (none) -> C22950
- R104: renamed from R116; footprint Resistor_SMD:R_0402_1005Metric -> Resistor_SMD:R_0603_1608Metric_Pad0.98x0.95mm_HandSolder; JLCPCB# (none) -> C23138
- R105: renamed from R109; footprint Resistor_SMD:R_0402_1005Metric -> Resistor_SMD:R_0603_1608Metric_Pad0.98x0.95mm_HandSolder; JLCPCB# (none) -> C23162
- R106: renamed from R111; footprint Resistor_SMD:R_0402_1005Metric -> Resistor_SMD:R_0603_1608Metric_Pad0.98x0.95mm_HandSolder; JLCPCB# (none) -> C23162
- R107: renamed from R117; footprint Resistor_SMD:R_0402_1005Metric -> Resistor_SMD:R_0603_1608Metric_Pad0.98x0.95mm_HandSolder; JLCPCB# (none) -> C22950
- R108: renamed from R118; footprint Resistor_SMD:R_0402_1005Metric -> Resistor_SMD:R_0603_1608Metric_Pad0.98x0.95mm_HandSolder; JLCPCB# (none) -> C23138
- R109: renamed from R113; footprint Resistor_SMD:R_0402_1005Metric -> Resistor_SMD:R_0603_1608Metric_Pad0.98x0.95mm_HandSolder; JLCPCB# C21190 -> C23162
- R110: renamed from R105; value Rg -> 820; footprint Resistor_SMD:R_0402_1005Metric -> Resistor_SMD:R_0603_1608Metric_Pad0.98x0.95mm_HandSolder; JLCPCB# (none) -> C23253
- R111: renamed from R101; value Rg -> 15k; footprint Resistor_SMD:R_0402_1005Metric -> Resistor_SMD:R_0603_1608Metric_Pad0.98x0.95mm_HandSolder; JLCPCB# (none) -> C22809
- R112: renamed from R107; value Rg -> 15k; footprint Resistor_SMD:R_0402_1005Metric -> Resistor_SMD:R_0603_1608Metric_Pad0.98x0.95mm_HandSolder; JLCPCB# (none) -> C22809
- R113: renamed from R108; value 11k -> 10k; footprint Resistor_SMD:R_0402_1005Metric -> Resistor_SMD:R_0603_1608Metric_Pad0.98x0.95mm_HandSolder; JLCPCB# (none) -> C25804
- R115: renamed from R104; value 11k -> 10k; footprint Resistor_SMD:R_0402_1005Metric -> Resistor_SMD:R_0603_1608Metric_Pad0.98x0.95mm_HandSolder; JLCPCB# (none) -> C25804
- R118: renamed from R106; footprint Resistor_SMD:R_0402_1005Metric -> Resistor_SMD:R_0603_1608Metric_Pad0.98x0.95mm_HandSolder; JLCPCB# (none) -> C23162
- SW101, SW102: footprint button:TS-1088-AR02016 -> Button_Switch_SMD:SW_SPST_TS-1088-xR020
- U101: renamed from U102; JLCPCB# (none) -> C473012
- U102: renamed from U103; footprint (none) -> Package_SO:SOIC-8_3.9x4.9mm_P1.27mm; JLCPCB# (none) -> C652556
- U103: renamed from U101; footprint (none) -> Package_SO:SOIC-8_3.9x4.9mm_P1.27mm; JLCPCB# (none) -> C652556
- U104: footprint (none) -> Package_SO:SOIC-8_3.9x4.9mm_P1.27mm; JLCPCB# (none) -> C652556
- renumbered C105 to C101, C107 to C102, C102 to C103, C103 to C104, C104 to C105, C101 to C106, C106 to C108
Connections:
- net +12V: now also J105.1 (Pin_1)
- net +3.3V: now also R103.1, J103.1 (Pin_1), J103.3 (Pin_3), J103.9 (Pin_9); no longer R103.2
- net +5V: now also C107.1, C109.1, C111.2, C112.2, C113.2, R114.1, R116.1, R121.1; no longer R113.1, R115.1
- net Base_Ref: now also R107.1; no longer R107.2
- net East_West_Ref: now also J103.4 (Pin_4), J103.7 (Pin_7)
- net Flash: now also C110.1
- net GND: now also R108.2, C107.2, C109.2, C110.2, C111.1, C112.1, C113.1, C114.1, C115.1, C116.1, C117.2, J103.12 (Pin_12), J103.6 (Pin_6), J103.8 (Pin_8), J105.2 (Pin_2), J105.4 (Pin_4), R119.2, R120.2, U105.10 (GND), U105.18 (GND), U105.26 (GND); no longer R108.1
- net Green_Wire: now also J103.10 (Pin_10)
- net North_South_Ref: now also J103.2 (Pin_2), J103.5 (Pin_5)
- net White_Wire: now also J103.11 (Pin_11)
- net at R104.2: now also R103.2; no longer R103.1
- net at U104.6 (Ref): now also C116.2, R117.2, R120.1
- net at R115.2, U103.6 (Ref): now also C115.2, R119.1
- net at R113.2, R118.1, U102.6 (Ref): now also C114.2
- new net: R117.1, R121.2
- new net: R115.1, R116.2
- new net: R113.1, R114.2
- new net: R107.2, R108.1
- new net +5V_panel: C117.1, J105.3 (Pin_3), U105.19 (VIN)
- no-connect marks 0 -> 8
Other:
- note added: ""Boot""
- note added: "Analog Sensors Anemometer Precipitation"
- note added: "Analog Sensors Instrumentation Amps"
- note added: "Double Check gain resistors"
- note added: "Microcontroller ESP32"
- note added: "Modem"
- note added: "PDN and Input Power"
- note added: "Precipitation Drainage Servo"
- note added: "Sensor Bus I2C Communication Bus"
- note added: "load_cell black_wire"
- note added: "load_cell red_wire"
- note removed: "Anemometer Strain Gauges"
- note removed: "ESP32"
- note removed: "Instrumentation Amps"
- note removed: "PDN"
- note removed: "Rain Gauge Loadcell"
- note removed: "Rain Gauge Servo Control"
- note removed: "Sensors I2C Communication Bus"
- title: Remote Weather Station -> Weather Station
- moved on the sheet: C101, C102, C108, J104, R103, R104, R107, R108, R110, R111, R112, R113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
