File: PCB/Remote_Weather_Station/Remote_Weather_Station.kicad_pcb (KiCad board)
At the start: 4 copper layers, 100 x 100 mm, 83 parts, among them J101 UART, J102 Stemma_QT_Connector, J103 wire_bus, J104 Servo_Connector, J105 power_in, SW101 SW_Push, SW102 SW_Push, U101 ESP32-WROOM-32D, U102 SIM7600X, U103 AD8227, U104 AD8227, U105 AD8227, U201 TPS561208DDCR, U202 AMS1117-3.3, U203 AMS1117-5.0, U204 TPS561201DDCR

Commit message: Added a few trace
Routing:
- net N_S_Value: track 0.00 -> 50.8 mm
- net E_W_Value: track 0.00 -> 50.4 mm, vias 0 -> 2
- net Rain_Value: track 0.00 -> 36.3 mm
- net GND: vias 48 -> 49
Changed lines of the file:
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@@
+	)
+	(via
+		(at 153.65 75.14)
+		(size 0.45)
+		(drill 0.3)
+		(layers "F.Cu" "B.Cu")
+		(net 2)
 	)
 	(via
@@
 	)
 	(segment
+		(start 154.92 75.12)
+		(end 154.9 75.1)
+		(width 0.25)
+		(layer "F.Cu")
+		(net 47)
+	)
+	(segment
+		(start 154.92 75.14)
+		(end 154.92 75.12)
+		(width 0.25)
+		(layer "F.Cu")
+		(net 47)
+	)
+	(via
+		(at 169 115.6)
+		(size 0.45)
+		(drill 0.3)
+		(layers "F.Cu" "B.Cu")
+		(net 47)
+	)
+	(via
+		(at 154.9 75.1)
+		(size 0.45)
+		(drill 0.3)
+		(layers "F.Cu" "B.Cu")
+		(net 47)
+	)
+	(segment
+		(start 166.1 115.6)
+		(end 169 115.6)
+		(width 0.25)
+		(layer "B.Cu")
+		(net 47)
+	)
+	(segment
+		(start 164.7 114.2)
+		(end 166.1 115.6)
+		(width 0.25)
+		(layer "B.Cu")
+		(net 47)
+	)
+	(segment
+		(start 154.9 76.5)
+		(end 158.8 80.4)
+		(width 0.25)
+		(layer "B.Cu")
+		(net 47)
+	)
+	(segment
+		(start 154.9 75.1)
+		(end 154.9 76.5)
+		(width 0.25)
+		(layer "B.Cu")
+		(net 47)
+	)
+	(segment
+		(start 158.8 80.4)
+		(end 162.7 80.4)
+		(width 0.25)
+		(layer "B.Cu")
+		(net 47)
+	)
+	(segment
+		(start 164.7 82.4)
+		(end 164.7 114.2)
+		(width 0.25)
+		(layer "B.Cu")
+		(net 47)
+	)
+	(segment
+		(start 162.7 80.4)
+		(end 164.7 82.4)
+		(width 0.25)
+		(layer "B.Cu")
+		(net 47)
+	)
+	(segment
+		(start 167 81.5)
+		(end 167 95.2)
+		(width 0.25)
+		(layer "F.Cu")
+		(net 51)
+	)
+	(segment
+		(start 151.9 77.7)
+		(end 163.2 77.7)
+		(width 0.25)
+		(layer "F.Cu")
+		(net 51)
+	)
+	(segment
+		(start 150.61 76.41)
+		(end 151.9 77.7)
+		(width 0.25)
+		(layer "F.Cu")
+		(net 51)
+	)
+	(segment
+		(start 171 99.2)
+		(end 171 107.6)
+		(width 0.25)
+		(layer "F.Cu")
+		(net 51)
+	)
+	(segment
+		(start 170.85 107.75)
+		(end 169 107.75)
+		(width 0.25)
+		(layer "F.Cu")
+		(net 51)
+	)
+	(segment
+		(start 171 107.6)
+		(end 170.85 107.75)
+		(width 0.25)
+		(layer "F.Cu")
+		(net 51)
+	)
+	(segment
+		(start 163.2 77.7)
+		(end 167 81.5)
+		(width 0.25)
+		(layer "F.Cu")
+		(net 51)
+	)
+	(segment
+		(start 150.61 73.89)
+		(end 150.61 76.41)
+		(width 0.25)
+		(layer "F.Cu")
+		(net 51)
+	)
+	(segment
+		(start 167 95.2)
+		(end 171 99.2)
+		(width 0.25)
+		(layer "F.Cu")
+		(net 51)
+	)
+	(segment
+		(start 152 73)
+		(end 152 76.3)
+		(width 0.25)
+		(layer "F.Cu")
+		(net 55)
+	)
+	(segment
+		(start 173.5 90.2)
+		(end 173.2 90.5)
+		(width 0.25)
+		(layer "F.Cu")
+		(net 55)
+	)
+	(segment
+		(start 163.8 76.9)
+		(end 173.5 86.6)
+		(width 0.25)
+		(layer "F.Cu")
+		(net 55)
+	)
+	(segment
+		(start 150.61 72.62)
+		(end 151.62 72.62)
+		(width 0.25)
+		(layer "F.Cu")
+		(net 55)
+	)
+	(segment
+		(start 173.5 86.6)
+		(end 173.5 90.2)
+		(width 0.25)
+		(layer "F.Cu")
+		(net 55)
+	)
+	(segment
+		(start 173.2 90.5)
+		(end 171.525 90.5)
+		(width 0.25)
+		(layer "F.Cu")
+		(net 55)
+	)
+	(segment
+		(start 151.62 72.62)
+		(end 152 73)
+		(width 0.25)
+		(layer "F.Cu")
+		(net 55)
+	)
+	(segment
+		(start 152 76.3)
+		(end 152.6 76.9)
+		(width 0.25)
+		(layer "F.Cu")
+		(net 55)
+	)
+	(segment
+		(start 152.6 76.9)
+		(end 163.8 76.9)
+		(width 0.25)
+		(layer "F.Cu")
+		(net 55)
+	)
+	(segment
