File: PCB/Remote_Weather_Station/Remote_Weather_Station.kicad_pcb (KiCad board)
At the start: 4 copper layers, 0 parts

Commit message: Add files via upload
Parts:
- added C101: 1u, Capacitor_SMD:C_0805_2012Metric, F.Cu at (176.0, 92.3)
- added C102: 1u, Capacitor_SMD:C_0805_2012Metric, F.Cu at (176.0, 95.3)
- added C103: 100n, Capacitor_SMD:C_0805_2012Metric, F.Cu at (176.0, 98.3)
- added C104: 1u, Capacitor_SMD:C_0805_2012Metric, F.Cu at (176.0, 101.3)
- added C105: 1u, Capacitor_SMD:C_0805_2012Metric, F.Cu at (176.0, 104.4)
- added C106: 1u, Capacitor_SMD:C_0805_2012Metric, F.Cu at (176.0, 107.4)
- added C107: 1u, Capacitor_SMD:C_0805_2012Metric, F.Cu at (180.5, 92.3)
- added C108: 1u, Capacitor_SMD:C_0805_2012Metric, F.Cu at (180.5, 95.3)
- added C109: 1u, Capacitor_SMD:C_0805_2012Metric, F.Cu at (180.5, 98.3)
- added C110: 1u, Capacitor_SMD:C_0805_2012Metric, F.Cu at (180.5, 101.3)
- added C111: 1u, Capacitor_SMD:C_0805_2012Metric, F.Cu at (180.5, 104.4)
- added C112: 1u, Capacitor_SMD:C_0805_2012Metric, F.Cu at (180.5, 107.4)
- added C113: 1u, Capacitor_SMD:C_0805_2012Metric, F.Cu at (184.9, 92.3)
- added C114: 1u, Capacitor_SMD:C_0805_2012Metric, F.Cu at (184.9, 95.3)
- added C115: 1u, Capacitor_SMD:C_0805_2012Metric, F.Cu at (184.9, 98.3)
- added C116: 1u, Capacitor_SMD:C_0805_2012Metric, F.Cu at (184.9, 101.3)
- added C117: 1u, Capacitor_SMD:C_0805_2012Metric, F.Cu at (184.9, 104.4)
- added C201: 100n, Capacitor_SMD:C_0805_2012Metric, F.Cu at (100.7, 155.7)
- added C202: 10u, Capacitor_SMD:C_0805_2012Metric, F.Cu at (100.7, 158.7)
- added C203: 10u, Capacitor_SMD:C_0805_2012Metric, F.Cu at (100.7, 161.7)
- added C204: 47u, Capacitor_SMD:C_1206_3216Metric, F.Cu at (120.0, 155.9)
- added C205: 10u, Capacitor_SMD:C_0805_2012Metric, F.Cu at (100.7, 164.8)
- added C206: 22u, Capacitor_SMD:C_1206_3216Metric, F.Cu at (120.0, 159.2)
- added C207: 10u, Capacitor_SMD:C_0805_2012Metric, F.Cu at (100.7, 167.8)
- added C208: 22u, Capacitor_SMD:C_1206_3216Metric, F.Cu at (120.0, 162.6)
- added C209: 100n, Capacitor_SMD:C_0805_2012Metric, F.Cu at (100.7, 170.8)
- added C210: 10u, Capacitor_SMD:C_0805_2012Metric, F.Cu at (100.7, 173.8)
- added C211: 10u, Capacitor_SMD:C_0805_2012Metric, F.Cu at (100.7, 176.8)
- added C212: 47u, Capacitor_SMD:C_1206_3216Metric, F.Cu at (120.0, 165.9)
- added D101: RED_LED, LED_SMD:LED_0603_1608Metric, F.Cu at (188.9, 125.5)
- added H101: MountingHole, MountingHole:MountingHole_2.7mm_M2.5, F.Cu at (151.5, 56.6)
- added H102: MountingHole, MountingHole:MountingHole_2.7mm_M2.5, F.Cu at (151.5, 63.5)
- added H103: MountingHole, MountingHole:MountingHole_2.7mm_M2.5, F.Cu at (151.5, 70.5)
- added H104: MountingHole, MountingHole:MountingHole_2.7mm_M2.5, F.Cu at (151.5, 77.4)
- added J101: UART, Connector_PinHeader_2.54mm:PinHeader_1x06_P2.54mm_Vertical, F.Cu at (184.5, 111.2)
- added J102: Stemma_QT_Connector, Connector_JST:JST_SH_BM04B-SRSS-TB_1x04-1MP_P1.00mm_Vertical, F.Cu at (191.3, 121.1)
- added J103: wire_bus, Terminal_Blocks:WJ250B-3.5-12P-11-00A, F.Cu at (164.9, 164.5)
- added J105: power_in, Terminal_Blocks:DBT50G-7.62-4P-BK-P, F.Cu at (106.5, 101.5)
- added L201: 4.7u, Inductor_SMD:L_Vishay_IFSC-1515AH_4x4x1.8mm, F.Cu at (110.1, 173.6)
- added L202: 4.7u, Inductor_SMD:L_Vishay_IFSC-1515AH_4x4x1.8mm, F.Cu at (110.1, 179.2)
- added R101: 680, Resistor_SMD:R_0603_1608Metric_Pad0.98x0.95mm_HandSolder, F.Cu at (162.9, 92.1)
- added R102: 4.7k, Resistor_SMD:R_0603_1608Metric_Pad0.98x0.95mm_HandSolder, F.Cu at (162.9, 94.6)
- added R103: 20, Resistor_SMD:R_0603_1608Metric_Pad0.98x0.95mm_HandSolder, F.Cu at (162.9, 97.1)
- added R104: 330, Resistor_SMD:R_0603_1608Metric_Pad0.98x0.95mm_HandSolder, F.Cu at (162.9, 99.6)
- added R105: 4.7k, Resistor_SMD:R_0603_1608Metric_Pad0.98x0.95mm_HandSolder, F.Cu at (162.9, 102.1)
- added R106: 4.7k, Resistor_SMD:R_0603_1608Metric_Pad0.98x0.95mm_HandSolder, F.Cu at (162.9, 104.6)
- added R107: 20, Resistor_SMD:R_0603_1608Metric_Pad0.98x0.95mm_HandSolder, F.Cu at (162.9, 107.1)
- added R108: 330, Resistor_SMD:R_0603_1608Metric_Pad0.98x0.95mm_HandSolder, F.Cu at (162.9, 109.6)
- added R109: 4.7k, Resistor_SMD:R_0603_1608Metric_Pad0.98x0.95mm_HandSolder, F.Cu at (167.3, 92.1)
- added R110: 820, Resistor_SMD:R_0603_1608Metric_Pad0.98x0.95mm_HandSolder, F.Cu at (167.3, 94.6)
- added R111: 15k, Resistor_SMD:R_0603_1608Metric_Pad0.98x0.95mm_HandSolder, F.Cu at (167.3, 97.1)
- added R112: 15k, Resistor_SMD:R_0603_1608Metric_Pad0.98x0.95mm_HandSolder, F.Cu at (167.3, 99.6)
- added R113: 10k, Resistor_SMD:R_0603_1608Metric_Pad0.98x0.95mm_HandSolder, F.Cu at (167.3, 102.1)
- added R114: 1k, Resistor_SMD:R_0603_1608Metric_Pad0.98x0.95mm_HandSolder, F.Cu at (167.3, 104.6)
- added R115: 10k, Resistor_SMD:R_0603_1608Metric_Pad0.98x0.95mm_HandSolder, F.Cu at (167.3, 107.1)
- added R116: 1k, Resistor_SMD:R_0603_1608Metric_Pad0.98x0.95mm_HandSolder, F.Cu at (167.3, 109.6)
- added R117: 10k, Resistor_SMD:R_0603_1608Metric_Pad0.98x0.95mm_HandSolder, F.Cu at (171.6, 92.1)
- added R118: 4.7k, Resistor_SMD:R_0603_1608Metric_Pad0.98x0.95mm_HandSolder, F.Cu at (171.6, 94.6)
- added R119: 4.7k, Resistor_SMD:R_0603_1608Metric_Pad0.98x0.95mm_HandSolder, F.Cu at (171.6, 97.1)
- added R120: 4.7k, Resistor_SMD:R_0603_1608Metric_Pad0.98x0.95mm_HandSolder, F.Cu at (171.6, 99.6)
- added R121: 1k, Resistor_SMD:R_0603_1608Metric_Pad0.98x0.95mm_HandSolder, F.Cu at (171.6, 102.1)
- added R201: 49.9k, Resistor_SMD:R_0603_1608Metric_Pad0.98x0.95mm_HandSolder, F.Cu at (105.1, 155.5)
- added R202: 10k, Resistor_SMD:R_0603_1608Metric_Pad0.98x0.95mm_HandSolder, F.Cu at (105.1, 158.0)
- added R203: 0, Resistor_SMD:R_0603_1608Metric_Pad0.98x0.95mm_HandSolder, F.Cu at (105.1, 160.5)
- added R204: 0, Resistor_SMD:R_0603_1608Metric_Pad0.98x0.95mm_HandSolder, F.Cu at (105.1, 163.0)
- added R205: 68k, Resistor_SMD:R_0603_1608Metric_Pad0.98x0.95mm_HandSolder, F.Cu at (105.1, 165.5)
- added R206: 10k, Resistor_SMD:R_0603_1608Metric_Pad0.98x0.95mm_HandSolder, F.Cu at (105.1, 168.0)
- added R207: 3.6k, Resistor_SMD:R_0603_1608Metric_Pad0.98x0.95mm_HandSolder, F.Cu at (105.1, 170.5)
- added SW101: SW_Push, Button_Switch_SMD:SW_SPST_TS-1088-xR020, F.Cu at (190.4, 111.2)
- added SW102: SW_Push, Button_Switch_SMD:SW_SPST_TS-1088-xR020, F.Cu at (190.4, 115.7)
- added U101: ESP32-WROOM-32D, RF_Module:ESP32-WROOM-32D, F.Cu at (131.6, 76.1)
- added U102: AD8227, Package_SO:SOIC-8_3.9x4.9mm_P1.27mm, F.Cu at (178.0, 112.2)
- added U103: AD8227, Package_SO:SOIC-8_3.9x4.9mm_P1.27mm, F.Cu at (178.0, 118.8)
- added U104: AD8227, Package_SO:SOIC-8_3.9x4.9mm_P1.27mm, F.Cu at (178.0, 125.4)
- added U105: SIM7600X, Modem_Footprint:SIM7600X, F.Cu at (137.3, 111.0)
- added U201: TPS561208DDCR, Package_TO_SOT_SMD:SOT-23-6, F.Cu at (115.5, 173.3)
- added U202: AMS1117-3.3, Package_TO_SOT_SMD:SOT-223-3_TabPin2, F.Cu at (112.2, 158.4)
- added U203: AMS1117-5.0, Package_TO_SOT_SMD:SOT-223-3_TabPin2, F.Cu at (112.2, 166.7)
- added U204: TPS561201DDCR, Package_TO_SOT_SMD:SOT-23-6, F.Cu at (115.5, 177.9)

Commit message: Add files via upload
Parts:
- added C106: 1u, Capacitor_SMD:C_0805_2012Metric, F.Cu at (89.7, 139.2)
- added C107: 1u, Capacitor_SMD:C_0805_2012Metric, F.Cu at (89.7, 142.2)
- added C120: 1u, Capacitor_SMD:C_0805_2012Metric, F.Cu at (89.7, 145.2)
- added C121: 1u, Capacitor_SMD:C_0805_2012Metric, F.Cu at (89.7, 148.2)
- added R102: 11k, Resistor_SMD:R_0603_1608Metric_Pad0.98x0.95mm_HandSolder, F.Cu at (94.1, 139.0)
- added R103: 11k, Resistor_SMD:R_0603_1608Metric_Pad0.98x0.95mm_HandSolder, F.Cu at (94.1, 141.5)
- added R124: 11k, Resistor_SMD:R_0603_1608Metric_Pad0.98x0.95mm_HandSolder, F.Cu at (94.1, 144.0)
- added R125: 11k, Resistor_SMD:R_0603_1608Metric_Pad0.98x0.95mm_HandSolder, F.Cu at (94.1, 146.5)
- moved U201 103.8 mm to (43.3, 98.7)
- moved U204 98.1 mm to (43.4, 111.4)
- moved L201 93.1 mm to (54.0, 99.4)
- moved C211 87.5 mm to (38.6, 115.1), turned to 180 degrees
- moved L202 87.5 mm to (53.9, 112.2)
- moved C203 87.4 mm to (38.6, 100.3), turned to 180 degrees
- moved C210 86.8 mm to (38.6, 113.1), turned to 180 degrees
- moved C202 83.9 mm to (38.6, 102.3), turned to 180 degrees
- moved C204 81.2 mm to (61.6, 99.5), turned to -90 degrees
- moved C209 79.8 mm to (48.0, 110.9)
- moved C212 79.3 mm to (61.8, 112.0), turned to -90 degrees
- moved C201 78.1 mm to (48.0, 98.1)
- moved R201 73.1 mm to (58.8, 98.9), turned to -90 degrees
- moved C205 73.1 mm to (64.5, 101.2), turned to -90 degrees
- moved R202 72.5 mm to (58.8, 102.2), turned to -90 degrees
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- renumbered C103 to C102, C104 to C103, C102 to C104, C106 to C108, C107 to C109, C108 to C110, C109 to C111, C110 to C112, C111 to C113, C112 to C114, C113 to C115, C117 to C116, C114 to C117, C115 to C118, C116 to C119, R102 to R104, R103 to R105, R104 to R106, R105 to R107, R106 to R108, R107 to R109, R108 to R110, R109 to R111, R110 to R112, R111 to R113, R112 to R114, R113 to R115, R114 to R116, R115 to R117, R116 to R118, R117 to R119, R121 to R120, R118 to R121, R119 to R122, R120 to R123, R207 to R206, R206 to R207, U105 to U102, U102 to U103, U103 to U104, U104 to U105
Connections:
- J102 pad MP: (no net) -> GND
- J103 pad 10: Green_Wire -> Green_Wire_in
- J103 pad 11: White_Wire -> White_Wire_in
- J103 pad 2: North_South_Ref -> /N_red_wire
- J103 pad 4: East_West_Ref -> /E_red_wire
- J103 pad 5: North_South_Ref -> /N_red_wire
- J103 pad 7: East_West_Ref -> /E_red_wire
- U103 pad 1: Green_Wire -> White_Wire
- U103 pad 4: White_Wire -> Green_Wire
Routing:
- net +12V: track 0.00 -> 21.2 mm
- net /PDN/6.3V_OUT: track 0.00 -> 18.7 mm
- net /PDN/4.6V_OUT: track 0.00 -> 18.6 mm
- net Net-(U204-VFB): track 0.00 -> 17.2 mm, vias 0 -> 2
- net Net-(U201-VFB): track 0.00 -> 15.9 mm, vias 0 -> 2
- net Net-(U201-SW): track 0.00 -> 11.2 mm, vias 0 -> 2
- net Net-(U204-SW): track 0.00 -> 11.0 mm, vias 0 -> 2
- net +5V: track 0.00 -> 8.70 mm, vias 0 -> 2
- net +3.3V: track 0.00 -> 8.70 mm, vias 0 -> 2
- net Net-(U201-VBST): track 0.00 -> 2.80 mm
- net Net-(U204-VBST): track 0.00 -> 2.69 mm
- net Net-(C208-Pad2): track 0.00 -> 1.65 mm
- net Net-(C206-Pad2): track 0.00 -> 1.65 mm
- net Net-(R205-Pad2): track 0.00 -> 1.50 mm
- net GND: vias 0 -> 16

Commit message: Add files via upload
Did a lot more of the layout. Still need vias
Parts:
- removed the R117 at (167.3, 107.1)
- removed the R118 at (167.3, 109.6)
- removed R119: 10k, Resistor_SMD:R_0603_1608Metric_Pad0.98x0.95mm_HandSolder
- removed R120: 1k, Resistor_SMD:R_0603_1608Metric_Pad0.98x0.95mm_HandSolder
- removed R122: 4.7k, Resistor_SMD:R_0603_1608Metric_Pad0.98x0.95mm_HandSolder
- removed the R123 at (171.6, 99.6)
- added C124: 1u, Capacitor_SMD:C_0805_2012Metric, F.Cu at (180.3, 101.6)
- added J104: Servo_Connector, Connector_PinHeader_2.54mm:PinHeader_1x03_P2.54mm_Vertical, F.Cu at (190.2, 143.5)
- R102, R103: value 11k -> 10k
- R112: renamed from R124; value 11k -> 10k
- R113: renamed from R125; value 11k -> 10k
- moved C113 108.0 mm to (179.5, 85.2)
- moved C114 104.8 mm to (179.4, 94.2)
- moved R112 102.7 mm to (179.5, 87.0), turned to 180 degrees
- moved R113 101.1 mm to (179.5, 92.5), turned to 180 degrees
- moved C106 93.1 mm to (175.0, 102.0), turned to 180 degrees
- moved C107 93.0 mm to (177.0, 110.2)
- moved H103 91.1 mm to (109.0, 151.0)
- moved R102 90.0 mm to (177.0, 104.0), turned to 180 degrees
- moved H104 88.7 mm to (201.0, 151.0)
- moved R103 87.9 mm to (177.0, 112.2), turned to 180 degrees
- moved C203 85.4 mm to (124.1, 99.8), turned to 90 degrees
- moved C202 83.4 mm to (122.0, 99.8), turned to 90 degrees
- moved U201 82.6 mm to (125.7, 104.4), turned to -90 degrees
- moved C201 79.0 mm to (126.3, 109.1), turned to -90 degrees
- moved C210 75.8 mm to (113.3, 99.8), turned to 90 degrees
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- renumbered C120 to C113, C121 to C114, C113 to C115, C114 to C116, C115 to C117, C116 to C118, C117 to C119, C118 to C120, C119 to C121, R112 to R114, R113 to R115, R114 to R116, R115 to R117, R116 to R118, R121 to R123
Connections:
- C105 pad 1: +5V -> +3.3V
- C119 pad 2: Net-(U103-Ref) -> /V_ref_amp
- C120 pad 2: Net-(U104-Ref) -> /V_ref_amp
- C121 pad 2: Net-(U105-Ref) -> /V_ref_amp
- J101 pad 1: +5V -> +3.3V
- J103 pad 10: Green_Wire_in -> /rain_white
- J103 pad 11: White_Wire_in -> /rain_green
- R112 pad 1: Green_Wire_in -> /rain_green
- R113 pad 1: White_Wire_in -> /rain_white
- R117 pad 2: Net-(U103-Ref) -> /V_ref_amp
- R123 pad 1: Net-(U103-Ref) -> /V_ref_amp
- U101 pad 11: unconnected-(U101-IO26-Pad11) -> modem_rx
- U101 pad 12: unconnected-(U101-IO27-Pad12) -> modem_tx
- U102 pad 21: unconnected-(U102-RXD-Pad21) -> modem_rx
- U102 pad 22: unconnected-(U102-TXD-Pad22) -> modem_tx
- U103 pad 6: Net-(U103-Ref) -> /V_ref_amp
- U104 pad 6: Net-(U104-Ref) -> /V_ref_amp
- U105 pad 6: Net-(U105-Ref) -> /V_ref_amp
Routing:
- net +3.3V: track 8.70 -> 65.6 mm
- net Flash: track 0.00 -> 42.3 mm, vias 0 -> 1
- net /N_red_wire: track 0.00 -> 39.8 mm
- net +5V_panel: track 0.00 -> 39.7 mm
- net /E_red_wire: track 0.00 -> 39.0 mm
- net TX: track 0.00 -> 36.9 mm, vias 0 -> 1
- net RX: track 0.00 -> 33.7 mm, vias 0 -> 1
- net Base_Ref: track 0.00 -> 29.3 mm, vias 0 -> 3
- net Reset: track 0.00 -> 21.1 mm
- net GND: track 0.00 -> 18.0 mm, vias 16 -> 24
- net /rain_green: track 0.00 -> 16.2 mm
- net /rain_white: track 0.00 -> 15.8 mm
- net +5V: track 8.70 -> 19.4 mm
- net /V_ref_amp: track 0.00 -> 8.70 mm
- net North_South_Ref: track 0.00 -> 4.97 mm
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- added copper zone on In2.Cu, net +12V
- added copper zone on In2.Cu, net +3.3V
- added copper zone on In2.Cu, net +5V
- added copper zone on In1.Cu, net GND
Other:
- board outline added: 100 x 100 mm

Commit message: Add files via upload
Parts:
- moved C118 41.1 mm to (162.2, 133.5), turned to 90 degrees
- moved U102 23.1 mm to (147.2, 140.7), turned to 180 degrees
Routing:
- net N_S_Value: track 0.00 -> 50.8 mm
- net E_W_Value: track 0.00 -> 50.4 mm, vias 0 -> 2
- net +5V_panel: track 39.7 -> 84.6 mm
- net Rain_Value: track 0.00 -> 36.3 mm
- net +3.3V: track 65.6 -> 96.4 mm, vias 2 -> 27
- net +5V: track 19.4 -> 43.1 mm, vias 2 -> 21
- net +12V: track 20.7 -> 31.8 mm, vias 0 -> 12
- net GND: vias 24 -> 49

Commit message: Add files via upload
Parts:
- moved D101 65.0 mm to (122.4, 61.0), turned to 0 degrees
- moved R101 61.4 mm to (126.4, 61.0), turned to 180 degrees
- moved R108 12.4 mm to (172.5, 63.7)
- moved R117 8.24 mm to (169.5, 125.1)
- moved R118 8.24 mm to (169.5, 128.6)
- moved R123 8.24 mm to (172.0, 124.2)
- moved C109 6.69 mm to (185.0, 142.7)
- moved R107 6.06 mm to (177.6, 59.9)
- moved J102 5.94 mm to (182.5, 146.3)
- moved C115 0.50 mm to (169.5, 119.5)
Connections:
- U101 pad 11: modem_rx -> modem_tx
- U101 pad 12: modem_tx -> modem_rx
- U101 pad 25: Flash -> Reset
Routing:
- net I2C-SCL: track 0.00 -> 126.6 mm, vias 0 -> 2
- net I2C-SDA: track 0.00 -> 115.9 mm
- net Servo: track 0.00 -> 110.3 mm, vias 0 -> 1
- net modem_tx: track 0.00 -> 88.5 mm, vias 0 -> 1
- net modem_rx: track 0.00 -> 82.8 mm, vias 0 -> 1
- net /V_ref_amp: track 8.70 -> 49.0 mm, vias 0 -> 2
- net +3.3V: track 96.4 -> 59.2 mm
- net GND: track 18.0 -> 2.96 mm
- net Net-(D101-A): track 0.00 -> 2.30 mm
- net +5V: track 43.1 -> 44.6 mm

Commit message: Add files via upload
Parts:
- moved C212 19.7 mm to (118.4, 103.7), turned to 90 degrees
- moved L202 8.07 mm to (118.7, 108.3), turned to 90 degrees
- moved D101 6.41 mm to (116.0, 61.0)
- moved R101 6.41 mm to (120.0, 61.0)
- moved J102 5.85 mm to (182.5, 152.2)
- moved C109 5.85 mm to (185.0, 148.5)
Connections:
- J101 pad 2: RX -> GND
- J101 pad 3: TX -> RX
- J101 pad 4: Reset -> TX
- J101 pad 5: Flash -> unconnected-(J101-Pin_5-Pad5)
- J101 pad 6: GND -> unconnected-(J101-Pin_6-Pad6)
- U101 pad 25: Reset -> Flash
Routing:
- net Flash: track 42.3 -> 8.00 mm, vias 1 -> 0
- net Net-(U204-VFB): track 17.2 -> 1.47 mm, vias 2 -> 0
- net Reset: track 21.1 -> 9.40 mm
- net I2C-SCL: track 126.6 -> 132.4 mm
- net I2C-SDA: track 115.9 -> 121.7 mm
- net Green_Wire: track 2.75 -> 4.52 mm
- net RX: track 33.7 -> 34.9 mm
- net TX: track 36.9 -> 37.8 mm
- net GND: track 2.96 -> 3.83 mm, vias 49 -> 51
Other:
- board text added: "+12V Panel V+"
- board text added: "+3.3V"
- board text added: "+5V Panel"
- board text added: "Antenna Side"
- board text added: "COW-Bois Remote Weather Station"
- board text added: "Panel GND"
- board text added: "PanelGND"
- board text added: "RX"
- board text added: "TX"
